File: rs485adapter/_autosave-rs485adapter.kicad_sch (KiCad schematic)
At the start: 7 parts

Commit message: schema
Other:
- moved on the sheet: J?
Changed lines of the file:
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@@
 	)
 	(no_connect
-		(at 64.77 73.66)
+		(at 44.45 76.2)
 	)
 	(no_connect
-		(at 64.77 76.2)
-	)
-	(wire
-		(pts
-			(xy 44.45 73.66) (xy 41.91 73.66)
-		)
-		(stroke
-			(width 0)
-			(type default)
-		)
-	)
-	(wire
-		(pts
-			(xy 41.91 71.12) (xy 41.91 73.66)
+		(at 44.45 78.74)
+	)
+	(wire
+		(pts
+			(xy 64.77 76.2) (xy 77.47 76.2)
 		)
 		(stroke
@@
 	(wire
 		(pts
-			(xy 41.91 76.2) (xy 41.91 78.74)
+			(xy 67.31 78.74) (xy 67.31 81.28)
 		)
 		(stroke
@@
 	(wire
 		(pts
+			(xy 77.47 76.2) (xy 77.47 87.63)
+		)
+		(stroke
+			(width 0)
+			(type default)
+		)
+	)
+	(wire
+		(pts
 			(xy 90.17 71.12) (xy 90.17 76.2)
 		)
@@
 	(wire
 		(pts
-			(xy 44.45 76.2) (xy 41.91 76.2)
-		)
-		(stroke
-			(width 0)
-			(type default)
-		)
-	)
-	(wire
-		(pts
-			(xy 77.47 76.2) (xy 77.47 87.63)
+			(xy 64.77 78.74) (xy 67.31 78.74)
 		)
 		(stroke
@@
 	(symbol
 		(lib_id "XT60PW-M:XT60PW-M")
-		(at 44.45 73.66 0)
+		(at 64.77 76.2 0)
+		(mirror y)
 		(unit 1)
 		(exclude_from_sim no)
@@
 		(fields_autoplaced yes)
 		(property "Reference" "J?"
-			(at 54.61 66.04 0)
+			(at 54.61 68.58 0)
 			(effects
 				(font
@@
 		)
 		(property "Value" "12V IN"
-			(at 54.61 68.58 0)
+			(at 54.61 71.12 0)
 			(effects
 				(font
@@
 		)
 		(property "Footprint" "XT60PWM"
-			(at 60.96 168.58 0)
+			(at 48.26 171.12 0)
 			(effects
 				(font
@@
 		)
 		(property "Datasheet" "https://www.tme.eu/Document/9b8d0c5eb7094295f3d3112c214d3ade/XT60PW%20SPEC.pdf"
-			(at 60.96 268.58 0)
+			(at 48.26 271.12 0)
 			(effects
 				(font
@@
 		)
 		(property "Description" "Socket; DC supply; XT60; male; PIN: 2; on PCBs; THT; Colour: yellow"
-			(at 44.45 73.66 0)
+			(at 64.77 76.2 0)
 			(effects
 				(font
@@
 		)
 		(property "Height" "8.4"
-			(at 60.96 468.58 0)
+			(at 48.26 471.12 0)
 			(effects
 				(font
@@
 		)
 		(property "Manufacturer_Name" "Changzou Amass Elec"
-			(at 60.96 568.58 0)
+			(at 48.26 571.12 0)
 			(effects
 				(font
@@
 		)
 		(property "Manufacturer_Part_Number" "XT60PW-M"
-			(at 60.96 668.58 0)
+			(at 48.26 671.12 0)
 			(effects
 				(font
@@
 		)
 		(property "Mouser Part Number" ""
-			(at 60.96 768.58 0)
+			(at 48.26 771.12 0)
 			(effects
 				(font
@@
 		)
 		(property "Mouser Price/Stock" ""
-			(at 60.96 868.58 0)
+			(at 48.26 871.12 0)
 			(effects
 				(font
@@
 		)
 		(property "Arrow Part Number" ""
-			(at 60.96 968.58 0)
+			(at 48.26 971.12 0)
 			(effects
 				(font
@@
 		)
 		(property "Arrow Price/Stock" ""
-			(at 60.96 1068.58 0)
+			(at 48.26 1071.12 0)
 			(effects
 				(font
@@
 	)
 	(symbol
-		(lib_id "power:+12V")
-		(at 41.91 71.12 0)
-		(unit 1)
-		(exclude_from_sim no)
-		(in_bom yes)
-		(on_board yes)
-		(dnp no)
-		(fields_autoplaced yes)
-		(property "Reference" "#PWR0101"
-			(at 41.91 74.93 0)
-			(effects
-				(font
-					(size 1.27 1.27)
-				)
-				(hide yes)
-			)
-		)
-		(property "Value" "+VINV"
-			(at 41.91 66.04 0)
-			(effects
-				(font
-					(size 1.27 1.27)
-				)
-			)
-		)
-		(property "Footprint" ""
-			(at 41.91 71.12 0)
-			(effects
-				(font
-					(size 1.27 1.27)
-				)
-				(hide yes)
-			)
-		)
-		(property "Datasheet" ""
-			(at 41.91 71.12 0)
-			(effects
-				(font
-					(size 1.27 1.27)
-				)
-				(hide yes)
-			)
-		)
-		(property "Description" "Power symbol creates a global label with name \"+12V\""
-			(at 41.91 71.12 0)
-			(effects
-				(font
-					(size 1.27 1.27)
-				)
-				(hide yes)
-			)
-		)
-		(pin "1"
-		)
-		(instances
-			(project "rs485adapter"
-				(path "/67070bee-4be5-4827-8b73-60c16857e4b5"
-					(reference "#PWR0101")
-					(unit 1)
-				)
-			)
-		)
-	)
-	(symbol
 		(lib_id "Connector:Conn_01x02_Pin")
 		(at 44.45 114.3 0)
@@
 	(symbol
 		(lib_id "power:GND")
-		(at 41.91 78.74 0)
+		(at 67.31 81.28 0)
+		(mirror y)
 		(unit 1)
 		(exclude_from_sim no)
@@
 		(fields_autoplaced yes)
 		(property "Reference" "#PWR0102"
-			(at 41.91 85.09 0)
+			(at 67.31 87.63 0)
 			(effects
 				(font
@@
 		)
 		(property "Value" "GND"
-			(at 41.91 83.82 0)
+			(at 67.31 86.36 0)
 			(effects
 				(font
@@
 		)
 		(property "Footprint" ""
-			(at 41.91 78.74 0)
+			(at 67.31 81.28 0)
 			(effects
 				(font
@@
 		)
 		(property "Datasheet" ""
-			(at 41.91 78.74 0)
+			(at 67.31 81.28 0)
 			(effects
 				(font
@@
 		)
 		(property "Description" "Power symbol creates a global label with name \"GND\" , ground"
-			(at 41.91 78.74 0)
-			(effects
-				(font
+			(at 67.31 81.28 0)
+			(effects
+				(font
