File: rs485adapter/psu.kicad_sch (KiCad schematic)
At the start: 10 parts

Commit message: bleugh
Parts:
- added C6, C7: 22u, Capacitor_SMD:C_1206_3216Metric, symbol Device:C
- C2: renamed from C?; footprint Capacitor_SMD:C_1206_3216Metric -> Capacitor_SMD:C_0603_1608Metric
- D4: renamed from D?; footprint (none) -> LED_SMD:LED_0603_1608Metric
- L1: renamed from L?; footprint (none) -> Inductor_SMD:L_Cenker_CKCS4030
- R10, R11, R9: renamed from R?; footprint (none) -> Resistor_SMD:R_0603_1608Metric
- gave numbers to parts that had none: 4
Connections:
- net +5V: now also C6.1, C7.1
- net GND: now also C6.2, C7.2
Other:
- moved on the sheet: C2, C3, C4, C5, D4, L1, R10, R11, R9, U2

Commit message: pushes
Parts:
- added C8: 22u, Capacitor_SMD:C_1210_3225Metric, symbol Device:C
- added C9: 100u, Capacitor_SMD:CP_Elec_5x3.9, symbol Device:C
- C2: footprint Capacitor_SMD:C_0603_1608Metric -> Capacitor_SMD:C_0805_2012Metric
- C3, C4, C5, C6, C7: footprint Capacitor_SMD:C_1206_3216Metric -> Capacitor_SMD:C_1210_3225Metric
- D4: footprint LED_SMD:LED_0603_1608Metric -> LED_SMD:LED_0805_2012Metric
- R10, R11, R9: footprint Resistor_SMD:R_0603_1608Metric -> Resistor_SMD:R_0805_2012Metric
Connections:
- net +12V: now also C4.1
- net +5V: now also C8.1, C9.1; no longer C4.1
- net GND: now also C8.2, C9.2
Other:
- moved on the sheet: C2, D4, L1, R10, R11, R9, U2
