File: rs485adapter/rs485.kicad_sch (KiCad schematic)
At the start: 11 parts

Commit message: schema
Parts:
- removed D? (x2): ESD131-B1-W0201, Diode_SMD:Infineon_SG-WLL-2-3_0.58x0.28_P0.36mm, symbol Diode:ESD131-B1-W0201
- removed F?: Fuse, symbol Device:Fuse
- removed JP?: SolderJumper_2_Open, symbol Jumper:SolderJumper_2_Open
- added D? (x2): ESD, Diode_SMD:D_SMA, symbol Diode:ESD131-B1-W0201
- added F?: Fuse, Fuse:Fuse_1812_4532Metric, symbol Device:Fuse
- added JP?: DE/RE SHORT, Jumper:SolderJumper-2_P1.3mm_Open_RoundedPad1.0x1.5mm, symbol Jumper:SolderJumper_2_Open
- added R? (x4): 10k, symbol Device:R
- D?: value ESD131-B1-W0201 -> ESD; footprint Diode_SMD:Infineon_SG-WLL-2-3_0.58x0.28_P0.36mm -> Diode_SMD:D_SMA
- F?: footprint (none) -> Fuse:Fuse_1812_4532Metric
- R? (x2): value R -> 10k
Connections:
- net E is gone; now on net GND: D?.1 (A1)
- net +5V: now also R?.1, R?.1, R?.1, R?.1
- net B-: now also F?.2
- net GND: now also D?.2 (A2)
- net at F?.1, R?.2, U?.6 (A): now also D?.1 (A1), D?.2 (A2)
- net RO: now reaches U?.1 (RO)
- net RO: now also R?.2
- net DE: now reaches U?.2 (~{RE})
- net DE: now also U?.3 (DE), JP?.1 (A), JP?.2 (B), R?.2, R?.2
- net DI: now reaches U?.4 (DI)
- net DI: now also R?.2
- net at D?.2 (A2), R?.1, U?.7 (B): now also D?.1 (A1), F?.1
Other:
- moved on the sheet: D?, F?, R?

Commit message: bleugh
Parts:
- C1: renamed from C?; footprint (none) -> Capacitor_SMD:C_0603_1608Metric
- R2, R3, R4, R5, R6, R7, R8: renamed from R?; footprint (none) -> Resistor_SMD:R_0603_1608Metric
- gave numbers to parts that had none: 7
Other:
- moved on the sheet: C1, D1, D2, D3, F1, F2, JP1, R2, R3, R4, R5, R6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

Commit message: pushes
Parts:
- removed D2: ESD, Diode_SMD:D_SMA, symbol Diode:ESD131-B1-W0201
- removed JP1: DE/RE SHORT, Jumper:SolderJumper-2_P1.3mm_Open_RoundedPad1.0x1.5mm, symbol Jumper:SolderJumper_2_Open
- C1: footprint Capacitor_SMD:C_0603_1608Metric -> Capacitor_SMD:C_0805_2012Metric
- R2, R3, R4, R5, R6, R7, R8: footprint Resistor_SMD:R_0603_1608Metric -> Resistor_SMD:R_0805_2012Metric
- renumbered D1 to D2, F1 to F2, F2 to F3
Connections:
- net A+: now also D2.2 (A2), R6.2
- net B-: now also D3.2 (A2), R8.1
- net DE: no longer R3.2, U1.2 (~{RE})
- net GND: now also D2.1 (A1); no longer D2.2 (A2)
- net at F2.1, U1.6 (A): no longer D2.1 (A1), R6.2
- net at F3.1, U1.7 (B): no longer D3.2 (A2), R8.1
- new net ¬RE: R3.2, U1.2 (~{RE})
Other:
- moved on the sheet: D2, D3, F2, F3, R7
