File: rs485adapter/rs485adapter.kicad_pcb (KiCad board)
At the start: 2 copper layers, 40 parts, among them J1 5V OUT, J2 XT60, J3 RACK OUT 2.54mm, J4 RACK OUT 2mm, J5 UART IN, J6 I2C OUT, U1 MAX485E, U2 AP62301WU, U3 INA219AxD

Commit message: pushes
Parts:
- removed JP1: DE/RE SHORT, Jumper:SolderJumper-2_P1.3mm_Open_RoundedPad1.0x1.5mm
- removed the R6 at (35.9, 98.6)
- removed the R8 at (35.9, 103.6)
- removed TP1: V-, TestPoint:TestPoint_Pad_2.0x2.0mm
- removed TP2: V+, TestPoint:TestPoint_Pad_2.0x2.0mm
- added C10: 100n, Capacitor_SMD:C_0805_2012Metric, F.Cu at (81.9, 59.1)
- added C9: 100u, Capacitor_SMD:CP_Elec_5x3.9, F.Cu at (90.8, 73.0)
- added F3: Fuse, Fuse:Fuse_1812_4532Metric, F.Cu at (84.3, 62.9)
- added H1: MountingHole, MountingHole:MountingHole_2.2mm_M2, F.Cu at (72.6, 59.5)
- added H2: MountingHole, MountingHole:MountingHole_2.2mm_M2, F.Cu at (83.8, 71.8)
- added R6: 10k, Resistor_SMD:R_0805_2012Metric, F.Cu at (85.8, 50.2)
- added R6: 10k, Resistor_SMD:R_0805_2012Metric, F.Cu at (85.8, 47.6)
- added R8: 10k, Resistor_SMD:R_0805_2012Metric, F.Cu at (85.8, 55.2)
- added R8: 10k, Resistor_SMD:R_0805_2012Metric, F.Cu at (85.8, 57.8)
- C1, C2: footprint Capacitor_SMD:C_0603_1608Metric -> Capacitor_SMD:C_0805_2012Metric
- C3, C4, C5, C6, C7: footprint Capacitor_SMD:C_1206_3216Metric -> Capacitor_SMD:C_1210_3225Metric
- C8: value 100n -> 22u; footprint Capacitor_SMD:C_0603_1608Metric -> Capacitor_SMD:C_1210_3225Metric
- D1: value ESD -> SBR3U60P1-7; footprint Diode_SMD:D_SMA -> Diode_SMD:D_PowerDI-123
- D4: footprint LED_SMD:LED_0603_1608Metric -> LED_SMD:LED_0805_2012Metric
- F1: value Fuse -> 3A
- J1: value 5V OUT -> VIN; footprint Connector_PinHeader_2.54mm:PinHeader_1x02_P2.54mm_Horizontal -> Connector_PinHeader_2.54mm:PinHeader_1x02_P2.54mm_Vertical
- J3: value RACK OUT 2.54mm -> RACK OUT 2mm; footprint Connector_PinHeader_2.54mm:PinHeader_1x06_P2.54mm_Horizontal -> Connector_PinHeader_2.00mm:PinHeader_1x06_P2.00mm_Vertical
- J4: value RACK OUT 2mm -> RACK OUT 2.54mm; footprint Connector_PinHeader_2.00mm:PinHeader_1x06_P2.00mm_Horizontal -> Connector_PinHeader_2.54mm:PinHeader_1x06_P2.54mm_Vertical
- J5: value UART IN -> IN/PWR 2.54mm; footprint Connector_PinHeader_2.54mm:PinHeader_1x04_P2.54mm_Horizontal -> Connector_PinHeader_2.54mm:PinHeader_1x08_P2.54mm_Vertical
- J6: value I2C OUT -> IN/PWR 2.00mm; footprint Connector_PinHeader_2.54mm:PinHeader_1x02_P2.54mm_Horizontal -> Connector_PinHeader_2.00mm:PinHeader_1x08_P2.00mm_Vertical
- R1, R10, R11, R12, R13, R2, R3, R4, R5, R7, R9: footprint Resistor_SMD:R_0603_1608Metric -> Resistor_SMD:R_0805_2012Metric
- moved R7 69.5 mm to (85.8, 52.7)
- moved D3 59.5 mm to (91.3, 62.9), turned to 180 degrees
- moved D2 54.9 mm to (91.3, 67.4), turned to 180 degrees
- moved D1 50.5 mm to (74.3, 48.3), turned to 180 degrees
- moved F1 43.6 mm to (74.7, 51.7)
- moved C3 43.4 mm to (80.6, 48.7), turned to 90 degrees
- moved F2 42.8 mm to (84.3, 67.3)
- moved C1 42.0 mm to (74.3, 68.9), turned to 90 degrees
- moved C4 41.7 mm to (80.6, 54.0), turned to -90 degrees
- moved J4 39.4 mm to (93.3, 45.7)
- moved U1 39.4 mm to (78.1, 70.2), turned to 90 degrees
- moved R2 37.9 mm to (70.5, 73.0), turned to 180 degrees
- moved R3 37.1 mm to (70.5, 77.5), turned to 180 degrees
- moved R4 37.1 mm to (70.5, 80.0), turned to 180 degrees
- moved R5 37.1 mm to (70.5, 82.5), turned to 180 degrees
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Connections:
- C4 pad 1: +5V -> +12V
- C8 pad 1: GND -> +5V
- C8 pad 2: +5V -> GND
- D1 pad 1: Net-(D1-A1) -> +VINV
- D2 pad 1: Net-(D2-A1) -> GND
- D2 pad 2: Net-(D1-A1) -> /A+
- D3 pad 2: Net-(D2-A1) -> /B-
- F1 pad 1: Net-(D1-A1) -> Net-(J1-Pin_2)
- F1 pad 2: /A+ -> +VINV
- F2 pad 1: Net-(D2-A1) -> Net-(U1-A)
- F2 pad 2: /B- -> /A+
- J1 pad 1: +5V -> GND
- J1 pad 2: GND -> Net-(J1-Pin_2)
- J2 pad 2: +VINV -> Net-(J1-Pin_2)
- J3 pad 5: unconnected-(J3-Pin_5-Pad5) -> /AUX1
- J3 pad 6: unconnected-(J3-Pin_6-Pad6) -> /AUX2
- J4 pad 5: unconnected-(J4-Pin_5-Pad5) -> /AUX1
- J4 pad 6: unconnected-(J4-Pin_6-Pad6) -> /AUX2
- J5 pad 1: /RO -> GND
- J5 pad 2: /DE -> +5V
- J5 pad 3: /DE -> /DI
- J5 pad 4: /DI -> /DE
- J6 pad 1: /SDA -> GND
- J6 pad 2: /SCL -> +5V
- R3 pad 2: /DE -> /¬RE
- U1 pad 2: /DE -> /¬RE
- U1 pad 6: Net-(D1-A1) -> Net-(U1-A)
- U1 pad 7: Net-(D2-A1) -> Net-(U1-B)
Routing:
- net +5V: track 0.00 -> 131.4 mm, vias 0 -> 5
- net +12V: track 0.00 -> 57.9 mm, vias 0 -> 6
- net GND: track 0.00 -> 43.6 mm, vias 0 -> 82
- net /A+: track 0.00 -> 30.6 mm
- net /DI: track 0.00 -> 27.1 mm
- net /SCL: track 0.00 -> 25.4 mm, vias 0 -> 2
- net /DE: track 0.00 -> 24.6 mm, vias 0 -> 2
- net /B-: track 0.00 -> 23.6 mm
- net /¬RE: track 0.00 -> 22.2 mm, vias 0 -> 2
- net /SDA: track 0.00 -> 21.4 mm, vias 0 -> 2
- net /RO: track 0.00 -> 17.1 mm
- net Net-(J1-Pin_2): track 0.00 -> 14.0 mm
- net Net-(U2-SW): track 0.00 -> 12.8 mm, vias 0 -> 2
- net +VINV: track 0.00 -> 12.1 mm
- net Net-(U1-B): track 0.00 -> 10.3 mm
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- added copper zone on B.Cu, net GND
- added copper zone on F.Cu, net GND
Other:
- board outline added: 34.3 x 42.2 mm
- board text added: "RS485 Tranciever & SMPS"
