File: rs485adapter/rs485adapter.kicad_sch (KiCad schematic)
At the start: 7 parts

Commit message: bleugh
Parts:
- removed J?: 12V IN, XT60PWM, symbol XT60PW-M:XT60PW-M
- added J2: XT60, Connector_AMASS:AMASS_XT60PW-F_1x02_P7.20mm_Horizontal, symbol Connector:Screw_Terminal_01x02
- added TP1: V-, TestPoint:TestPoint_Pad_2.0x2.0mm, symbol Connector:TestPoint
- added TP2: V+, TestPoint:TestPoint_Pad_2.0x2.0mm, symbol Connector:TestPoint
- J1, J6: renamed from J?; footprint (none) -> Connector_PinHeader_2.54mm:PinHeader_1x02_P2.54mm_Horizontal
- J3: renamed from J?; footprint (none) -> Connector_PinHeader_2.54mm:PinHeader_1x06_P2.54mm_Horizontal
- J4: renamed from J?; footprint (none) -> Connector_PinHeader_2.00mm:PinHeader_1x06_P2.00mm_Horizontal
- J5: renamed from J?; footprint (none) -> Connector_PinHeader_2.54mm:PinHeader_1x04_P2.54mm_Horizontal
- R1: renamed from R?; footprint (none) -> Resistor_SMD:R_0603_1608Metric
Connections:
- net +12V: now also J3.1 (Pin_1), J4.1 (Pin_1)
- net +VINV: now also J2.2 (Pin_2), TP2.1
- net GND: now also J1.2 (Pin_2), J3.2 (Pin_2), J4.2 (Pin_2), J2.1 (Pin_1), TP1.1
- net RO: now reaches J5.1 (Pin_1)
- net ¬RE: now reaches J5.2 (Pin_2)
- net DE: now reaches J5.3 (Pin_3)
- net DI: now reaches J5.4 (Pin_4)
- net SDA: now reaches J6.1 (Pin_1)
- net SCL: now reaches J6.2 (Pin_2)
- net A+: now reaches J3.3 (Pin_3)
- net A+: now also J4.3 (Pin_3)
- net B-: now reaches J3.4 (Pin_4)
- net B-: now also J4.4 (Pin_4)
- net +5V: now reaches J1.1 (Pin_1)
- no-connect marks 2 -> 4
Other:
- note removed: "output to exactly the mount connctor"
- moved on the sheet: J1, J3, J4, J5, J6, R1

Commit message: pushes
Parts:
- removed J5: UART IN, Connector_PinHeader_2.54mm:PinHeader_1x04_P2.54mm_Horizontal, symbol Connector:Conn_01x04_Pin
- removed J6: I2C OUT, Connector_PinHeader_2.54mm:PinHeader_1x02_P2.54mm_Horizontal, symbol Connector:Conn_01x02_Pin
- removed TP1: V-, TestPoint:TestPoint_Pad_2.0x2.0mm, symbol Connector:TestPoint
- removed TP2: V+, TestPoint:TestPoint_Pad_2.0x2.0mm, symbol Connector:TestPoint
- added D1: SBR3U60P1-7, Diode_SMD:D_PowerDI-123, symbol Device:D_Schottky
- added F1: 3A, Fuse:Fuse_1812_4532Metric, symbol Device:Fuse
- added H1, H2: MountingHole, MountingHole:MountingHole_2.2mm_M2, symbol Mechanical:MountingHole
- added J5: IN/PWR 2.54mm, Connector_PinHeader_2.54mm:PinHeader_1x08_P2.54mm_Vertical, symbol Connector:Conn_01x08_Pin
- added J6: IN/PWR 2.00mm, Connector_PinHeader_2.00mm:PinHeader_1x08_P2.00mm_Vertical, symbol Connector:Conn_01x08_Pin
- J1: value 5V OUT -> VIN; footprint Connector_PinHeader_2.54mm:PinHeader_1x02_P2.54mm_Horizontal -> Connector_PinHeader_2.54mm:PinHeader_1x02_P2.54mm_Vertical
- J3: renamed from J4; footprint Connector_PinHeader_2.00mm:PinHeader_1x06_P2.00mm_Horizontal -> Connector_PinHeader_2.00mm:PinHeader_1x06_P2.00mm_Vertical
- J4: renamed from J3; footprint Connector_PinHeader_2.54mm:PinHeader_1x06_P2.54mm_Horizontal -> Connector_PinHeader_2.54mm:PinHeader_1x06_P2.54mm_Vertical
- R1: footprint Resistor_SMD:R_0603_1608Metric -> Resistor_SMD:R_0805_2012Metric
Connections:
- net +5V: now also J5.2 (Pin_2), J6.2 (Pin_2); no longer J1.1 (Pin_1)
- net +VINV: now also D1.1 (K), F1.2; no longer J2.2 (Pin_2)
- net DE: now also J5.4 (Pin_4), J6.4 (Pin_4)
- net DI: now also J5.3 (Pin_3), J6.3 (Pin_3)
- net GND: now also J1.1 (Pin_1), D1.2 (A), J5.1 (Pin_1), J6.1 (Pin_1); no longer J1.2 (Pin_2)
- net RO: now also J5.6 (Pin_6), J6.6 (Pin_6)
- net SCL: now also J5.7 (Pin_7), J6.7 (Pin_7)
- net SDA: now also J5.8 (Pin_8), J6.8 (Pin_8)
- net ¬RE: now also J5.5 (Pin_5), J6.5 (Pin_5)
- net AUX1: now reaches J4.5 (Pin_5)
- net AUX1: now also J3.5 (Pin_5)
- net AUX2: now reaches J4.6 (Pin_6)
- net AUX2: now also J3.6 (Pin_6)
- new net: F1.1, J1.2 (Pin_2), J2.2 (Pin_2)
- no-connect marks 4 -> 0
Other:
- moved on the sheet: J2, J3, J4, R1
