File: rs485adapter/sense.kicad_sch (KiCad schematic)
At the start: 4 parts

Commit message: bleugh
Parts:
- C8: renamed from C?; footprint (none) -> Capacitor_SMD:C_0603_1608Metric
- R12, R13: renamed from R?; footprint (none) -> Resistor_SMD:R_0603_1608Metric
- gave numbers to parts that had none: 1
Other:
- moved on the sheet: C8, R12, R13, U3

Commit message: pushes
Parts:
- C10: renamed from C8; footprint Capacitor_SMD:C_0603_1608Metric -> Capacitor_SMD:C_0805_2012Metric
- R12, R13: footprint Resistor_SMD:R_0603_1608Metric -> Resistor_SMD:R_0805_2012Metric
Changed lines of the file:
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@@
 		(dnp no)
 		(fields_autoplaced yes)
-		(property "Reference" "#PWR035"
+		(property "Reference" "#PWR040"
 			(at 116.84 91.44 0)
 			(effects
@@
 			(project "rs485adapter"
 				(path "/67070bee-4be5-4827-8b73-60c16857e4b5/5c441b0c-0b61-424c-828d-9cbeb3302948"
-					(reference "#PWR035")
+					(reference "#PWR040")
 					(unit 1)
 				)
@@
 			)
 		)
-		(property "Footprint" "Resistor_SMD:R_0603_1608Metric"
+		(property "Footprint" "Resistor_SMD:R_0805_2012Metric"
 			(at 135.128 54.61 90)
 			(effects
@@
 		(dnp no)
 		(fields_autoplaced yes)
-		(property "Reference" "#PWR031"
+		(property "Reference" "#PWR036"
 			(at 124.46 50.8 0)
 			(effects
@@
 			(project "rs485adapter"
 				(path "/67070bee-4be5-4827-8b73-60c16857e4b5/5c441b0c-0b61-424c-828d-9cbeb3302948"
-					(reference "#PWR031")
+					(reference "#PWR036")
 					(unit 1)
 				)
@@
 			)
 		)
-		(property "Footprint" "Resistor_SMD:R_0603_1608Metric"
+		(property "Footprint" "Resistor_SMD:R_0805_2012Metric"
 			(at 126.238 54.61 90)
 			(effects
@@
 		(dnp no)
 		(fields_autoplaced yes)
-		(property "Reference" "#PWR032"
+		(property "Reference" "#PWR037"
 			(at 133.35 50.8 0)
 			(effects
@@
 			(project "rs485adapter"
 				(path "/67070bee-4be5-4827-8b73-60c16857e4b5/5c441b0c-0b61-424c-828d-9cbeb3302948"
-					(reference "#PWR032")
+					(reference "#PWR037")
 					(unit 1)
 				)
@@
 		(dnp no)
 		(fields_autoplaced yes)
-		(property "Reference" "C8"
+		(property "Reference" "C10"
 			(at 96.52 43.18 90)
 			(effects
@@
 			)
 		)
-		(property "Footprint" "Capacitor_SMD:C_0603_1608Metric"
+		(property "Footprint" "Capacitor_SMD:C_0805_2012Metric"
 			(at 100.33 49.8348 0)
 			(effects
@@
 			(project "rs485adapter"
 				(path "/67070bee-4be5-4827-8b73-60c16857e4b5/5c441b0c-0b61-424c-828d-9cbeb3302948"
-					(reference "C8")
+					(reference "C10")
 					(unit 1)
 				)
@@
 		(dnp no)
 		(fields_autoplaced yes)
-		(property "Reference" "#PWR030"
+		(property "Reference" "#PWR035"
 			(at 104.14 50.8 0)
 			(effects
@@
 			(project "rs485adapter"
 				(path "/67070bee-4be5-4827-8b73-60c16857e4b5/5c441b0c-0b61-424c-828d-9cbeb3302948"
-					(reference "#PWR030")
+					(reference "#PWR035")
 					(unit 1)
 				)
@@
 		(dnp no)
 		(fields_autoplaced yes)
-		(property "Reference" "#PWR033"
+		(property "Reference" "#PWR038"
 			(at 88.9 60.96 0)
 			(effects
@@
 			(project "rs485adapter"
 				(path "/67070bee-4be5-4827-8b73-60c16857e4b5/5c441b0c-0b61-424c-828d-9cbeb3302948"
-					(reference "#PWR033")
+					(reference "#PWR038")
 					(unit 1)
 				)
@@
 		(dnp no)
 		(fields_autoplaced yes)
-		(property "Reference" "#PWR034"
+		(property "Reference" "#PWR039"
 			(at 104.14 91.44 0)
 			(effects
@@
 			(project "rs485adapter"
 				(path "/67070bee-4be5-4827-8b73-60c16857e4b5/5c441b0c-0b61-424c-828d-9cbeb3302948"
-					(reference "#PWR034")
-					(unit 1)
-				)
+					(reference "#PWR039")
+					(unit 1)
+				)
