File: rs485adaptershield/shield.kicad_pcb (KiCad board)
At the start: 4 copper layers, 66 x 53.3 mm, 106 parts, among them IC1 USB2422-I_MJ, IC2 THVD1406DRLR, J2 XT60, J7 RACK OUT 2.00mm, Q3 UT6KE5, U1 INA293B3, U10 TPSM33606S5QRDNRQ1, U11 MCP9700Ax-ETT, U2 Analog_1, U3 Analog_2, U5 TPSM33606S5QRDNRQ1, U6 Digital_1, U7 Digital_2, U8 AP2171W, U9 AP2171W, U901 USBLC6-2SC6, U902 USBLC6-2SC6, Y1 SG-210STF

Commit message: pushes
Parts:
- moved R19 16.8 mm to (114.0, 74.5)
- moved R16 14.5 mm to (162.7, 112.0)
- moved R23 14.5 mm to (163.7, 112.0)
- moved R14 14.5 mm to (162.7, 97.5)
- moved R15 14.5 mm to (163.7, 97.5)
- moved D7 7.72 mm to (166.0, 78.7), turned to 180 degrees
- moved C12 3.99 mm to (114.0, 72.5)
- moved R38 3.99 mm to (114.0, 73.5)
- moved R11 1.65 mm to (114.5, 113.2)
- moved D5 1.60 mm to (114.5, 111.6)
- moved R39 1.04 mm to (150.7, 73.0)
- moved R37 1.00 mm to (151.7, 73.0)
Connections:
- net /RS485 TxRx/¬RE renamed /RS485 TxRx/¬RESET
- net /RS485 TxRx/¬SHDN renamed /RS485 TxRx/¬SHUTDOWN
- net Net-(IC2-D) renamed /RS485 TxRx/TX
- C32 pad 1: Net-(J7-Pin_6) -> VBATT
- C40 pad 1: Net-(J7-Pin_6) -> VBATT
- IC2 pad 1: /RS485 TxRx/R -> /RS485 TxRx/RX
- R11 pad 1: /Current and Temp Sense/R_SENSE+ -> VBATT
- R33 pad 2: /RS485 TxRx/R -> /RS485 TxRx/RX
- R41 pad 2: /RS485 TxRx/R -> /RS485 TxRx/RX
- U7 pad 11: /USB_PSU_EN -> /USB_HUB_RST
- U7 pad 12: /¬USB_HUB_RST -> /USB_PWR_SHDN
Routing:
- net /RS485 TxRx/¬RESET: track 0.00 -> 26.7 mm, vias 0 -> 2
- net VBATT: track 0.00 -> 24.7 mm, vias 0 -> 8
- net Net-(J6-SHIELD): track 0.00 -> 23.0 mm
- net Net-(J1-SHIELD): track 0.00 -> 21.6 mm
- net Net-(J5-SHIELD): track 0.00 -> 21.6 mm
- net /RS485 TxRx/RX: track 0.00 -> 18.5 mm
- net /USB/EN_A: track 0.00 -> 17.8 mm
- net /RS485 TxRx/R: track 0.00 -> 17.2 mm
- net /RS485 TxRx/D: track 0.00 -> 16.2 mm
- net /RS485 TxRx/TX: track 0.00 -> 15.8 mm
- net /A: track 0.00 -> 15.8 mm
- net /USB/¬FLG_A: track 0.00 -> 15.2 mm
- net /B: track 0.00 -> 15.1 mm
- net /USB_PWR_SHDN: track 0.00 -> 12.8 mm
- net /RS485 TxRx/¬SHUTDOWN: track 0.00 -> 9.87 mm, vias 0 -> 2
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- added copper zone on In2.Cu, net VBATT
- removed copper zone on In2.Cu, net GND

Commit message: more layout
Parts:
- U10, U5: footprint IMPORTED:RDN0011A_TEX -> IMPORTED:RDN0011A_TEX_NEW
- moved TP7 89.2 mm to (169.0, 106.7)
- moved TP6 84.4 mm to (169.0, 92.2)
- moved TP5 66.2 mm to (143.3, 98.4)
- moved TP9 63.8 mm to (142.9, 88.9)
- moved TP8 57.5 mm to (142.9, 78.2)
- moved TP2 56.4 mm to (131.9, 72.3)
- moved TP4 50.6 mm to (143.4, 80.6)
- moved TP1 43.9 mm to (131.9, 83.0)
- moved C3 13.4 mm to (133.6, 79.3)
- moved C7 13.4 mm to (140.0, 74.9)
- moved C8 13.4 mm to (142.9, 74.9)
- moved U5 13.4 mm to (135.6, 74.9)
- moved C9 13.4 mm to (134.4, 77.7)
- moved C10 13.4 mm to (134.5, 71.8)
- moved C39 13.4 mm to (137.3, 77.8)
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Connections:
- net /DA+ renamed /DB _P
- net /DA- renamed /DB_N
- net /DB+ renamed /DA_P
- net /DB- renamed /DA_N
- net /DCONN_1+ renamed Net-(J1-D+-PadA6)
- net /DCONN_1- renamed Net-(J1-D--PadA7)
- net /DCONN_2+ renamed Net-(J5-D+-PadA6)
- net /DCONN_2- renamed Net-(J5-D--PadA7)
- net /DI+ renamed /DI_P
- net /DI- renamed /DI_N
- net VUSB1 renamed VUSB_B
- net VUSB2 renamed VUSB_A
- C21 pad 2: +5V -> +3.3V
- IC2 pad 8: +5V -> +3.3V
- J1 pad A4: /VBUS_OUT_A -> /VBUS_OUT_B
- J1 pad A5: /USB_CC1A -> /USB_CC1B
- J1 pad A9: /VBUS_OUT_A -> /VBUS_OUT_B
- J1 pad B4: /VBUS_OUT_A -> /VBUS_OUT_B
- J1 pad B5: /USB_CC2A -> /USB_CC2B
- J1 pad B9: /VBUS_OUT_A -> /VBUS_OUT_B
- J5 pad A4: /VBUS_OUT_B -> /VBUS_OUT_A
- J5 pad A5: /USB_CC1B -> /USB_CC1A
- J5 pad A9: /VBUS_OUT_B -> /VBUS_OUT_A
- J5 pad B4: /VBUS_OUT_B -> /VBUS_OUT_A
- J5 pad B5: /USB_CC2B -> /USB_CC2A
- J5 pad B9: /VBUS_OUT_B -> /VBUS_OUT_A
- R10 pad 1: /VBUS_OUT_B -> /VBUS_OUT_A
- R14 pad 1: /USB_CC2A -> /USB_CC2B
- R14 pad 2: /VBUS_A -> /VBUS_OUT_B
- R15 pad 1: /USB_CC1A -> /USB_CC1B
- R15 pad 2: /VBUS_A -> /VBUS_OUT_B
- R16 pad 1: /USB_CC2B -> /USB_CC2A
- R16 pad 2: /VBUS_B -> /VBUS_OUT_A
- R23 pad 1: /USB_CC1B -> /USB_CC1A
- R23 pad 2: /VBUS_B -> /VBUS_OUT_A
- R29 pad 1: /VBUS_OUT_A -> /VBUS_OUT_B
- R33 pad 1: +5V -> +3.3V
- R37 pad 1: +5V -> +3.3V
- U901 pad 5: /VBUS_OUT_A -> /VBUS_OUT_B
- U902 pad 5: /VBUS_OUT_B -> /VBUS_OUT_A
Routing:
- net +3.3V: track 15.1 -> 123.0 mm, vias 0 -> 6
- net GND: track 4.62 -> 41.5 mm, vias 0 -> 42
- net VUSB_B: track 0.00 -> 35.8 mm, vias 0 -> 3
- net Net-(U1-OUT): track 0.00 -> 34.6 mm, vias 0 -> 2
- net /USB_PSU_EN: track 0.94 -> 33.7 mm, vias 0 -> 2
- net VUSB_A: track 0.00 -> 30.7 mm, vias 0 -> 3
- net /¬USB_HUB_RST: track 5.48 -> 34.7 mm, vias 0 -> 5
- net VBATT: track 24.7 -> 39.5 mm, vias 8 -> 15
- net /VBUS_OUT_B: track 0.00 -> 12.0 mm, vias 0 -> 11
- net /VBUS_OUT_A: track 0.00 -> 10.3 mm, vias 0 -> 11
- net /VBUS_IN: track 7.37 -> 14.8 mm
- net /USB/EN_A: track 17.8 -> 11.9 mm, vias 0 -> 2
- net /Power Supply/FB2: track 0.00 -> 5.05 mm, vias 0 -> 1
- net /Power Supply/FB1: track 0.00 -> 5.05 mm, vias 0 -> 1
- net /USB/¬FLG_A: track 15.2 -> 11.8 mm, vias 0 -> 2
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- added copper zone on In2.Cu, net /VBUS_OUT_A
- added copper zone on In2.Cu, net /VBUS_OUT_B
