File: rs485adaptershield/shield.kicad_sch (KiCad schematic)
At the start: 35 parts, among them J2 XT60, J7 RACK OUT 2.00mm, Q3 UT6KE5, U2 Analog_1, U3 Analog_2, U6 Digital_1, U7 Digital_2, U901 USBLC6-2SC6, U902 USBLC6-2SC6

Commit message: more layout
Parts:
- added TP10: 5V, TestPoint:TestPoint_Pad_D1.0mm, symbol Connector:TestPoint
Connections:
- net VBUS_A is gone; now on net VBUS_OUT_B: R14.2, R15.2
- net VBUS_B is gone; now on net VBUS_OUT_A: R16.2, R23.2
- net DA_N: now also U902.6 (I/O1); no longer U901.6 (I/O1)
- net DA_P: now also U902.4 (I/O2); no longer U901.4 (I/O2)
- net DB _P: now also U901.4 (I/O2); no longer U902.4 (I/O2)
- net DB_N: now also U901.6 (I/O1); no longer U902.6 (I/O1)
- net USB_CC1A: now also J5.A5 (CC1), R23.1; no longer J1.A5 (CC1), R15.1
- net USB_CC1B: now also J1.A5 (CC1), R15.1; no longer J5.A5 (CC1), R23.1
- net USB_CC2A: now also J5.B5 (CC2), R16.1; no longer J1.B5 (CC2), R14.1
- net USB_CC2B: now also J1.B5 (CC2), R14.1; no longer J5.B5 (CC2), R16.1
- net VBUS_OUT_A: now also J5.A4 (VBUS), J5.A9 (VBUS), J5.B4 (VBUS), J5.B9 (VBUS), U902.5 (VBUS); no longer J1.A4 (VBUS), J1.A9 (VBUS), J1.B4 (VBUS), J1.B9 (VBUS), U901.5 (VBUS)
- net VBUS_OUT_B: now also J1.A4 (VBUS), J1.A9 (VBUS), J1.B4 (VBUS), J1.B9 (VBUS), U901.5 (VBUS); no longer J5.A4 (VBUS), J5.A9 (VBUS), J5.B4 (VBUS), J5.B9 (VBUS), U902.5 (VBUS)
- net +5V: no longer names the net of U2.5 (+5V)
- net +5V: now also TP10.1
Other:
- sheet USB ports: added USB_OUT_VBUS_A, USB_OUT_VBUS_B; removed USB_OUT1_VBUS, USB_OUT2_VBUS
- note removed: "5V Domain"
- moved on the sheet: J7, R14, R15, R16, R23
